File: gcm0/jinshu/kicad/jinshutance.sch (KiCad schematic (older format))
At the start: 51 parts, among them U1 LM317_TO3, U2 LM2596T-ADJ, U3 LM1117-3.3, U5 STM32F030F4P6, U6 TL084

Commit message: 探测金属管道缝隙成功
Parts:
- removed Q?: BC547, Package_TO_SOT_THT:TO-92_Inline, symbol Transistor_BJT:BC547
- removed Q?: BC557, Package_TO_SOT_THT:TO-92_Inline, symbol Transistor_BJT:BC557
- added D2: LED, symbol Device:LED
- added Q1: S8050, Package_TO_SOT_THT:TO-92_Inline, symbol Transistor_BJT:S8050
- added Q2: S8550, Package_TO_SOT_THT:TO-92_Inline, symbol Transistor_BJT:S8550
- added R17: 1K, symbol Device:R
- added SW1: SW_Push, symbol Switch:SW_Push
- added unit 2 of U4
- R13: value 510 -> 500
- R18: renamed from R?; value 500 -> 100
- R19: renamed from R?; value 33.3 -> 10
- gave numbers to parts that had none: 12
Connections:
- net +5: now also Q1.3 (C)
- net -5: now also Q2.3 (C)
- net GND: now also D2.1 (K), SW1.2
- net adc: now also U5.10 (PA4)
- net at U5.11 (PA5): now also SW1.1
- net at U5.12 (PA6): now also R17.2
- net at R15.1, U6.7: now also U4.5 (+); no longer R13.2
- net at R19.1, U4.2 (-): now also Q1.1 (E), Q2.1 (E)
- net at R18.1: now also Q1.2 (B), Q2.2 (B)
- net ADC: no longer names the net of U5.6 (PA0)
- new net: R13.2, U4.6 (-), U4.7
- new net: D2.2 (A), R17.1
Other:
- moved on the sheet: C16, R13

Commit message: 按键校0
Parts:
- Q1: value S8050 -> SS8050
- Q2: value S8550 -> SS8550
Changed lines of the file:
@@
 P 9550 4150
 F 0 "Q2" H 9740 4196 50  0000 L CNN
-F 1 "S8550" H 9740 4105 50  0000 L CNN
+F 1 "SS8550" H 9740 4105 50  0000 L CNN
 F 2 "Package_TO_SOT_THT:TO-92_Inline" H 9750 4075 50  0001 L CIN
 F 3 "http://www.unisonic.com.tw/datasheet/S8550.pdf" H 9550 4150 50  0001 L CNN
@@
 P 9550 3650
 F 0 "Q1" H 9740 3696 50  0000 L CNN
-F 1 "S8050" H 9740 3605 50  0000 L CNN
+F 1 "SS8050" H 9740 3605 50  0000 L CNN
 F 2 "Package_TO_SOT_THT:TO-92_Inline" H 9750 3575 50  0001 L CIN
 F 3 "http://www.unisonic.com.tw/datasheet/S8050.pdf" H 9550 3650 50  0001 L CNN
