File: gcm0/jiaodu_chuanganqi/kicad/Resolver.sch (KiCad schematic (older format))
At the start: 76 parts, among them Q1 S8050, Q2 S8550, Q3 BC547, U4 STM32F030F4P6, U6 TL084, U7 TL084, U8 NE5532, Y1 8MHZ

Commit message: 画了PCB
Parts:
- removed C21, C22: 2.2uF, symbol Device:CP
- removed D3, D4: LED, symbol Device:LED
- removed L1, L2, L4, L5: 200t, symbol Device:L_Core_Ferrite
- removed L3: 20t, symbol Device:L_Core_Ferrite
- removed L6: 20t, symbol Device:L
- removed L7: 200t, symbol Device:L
- removed Q3: BC547, Package_TO_SOT_THT:TO-92_Inline, symbol Transistor_BJT:BC547
- removed R25: 1K, symbol Device:R
- added C13: 105, Capacitor_SMD:C_0805_2012Metric_Pad1.18x1.45mm_HandSolder, symbol Device:C
- added C21, C22: 102, Capacitor_THT:C_Disc_D7.5mm_W5.0mm_P10.00mm, symbol Device:C
- added J1, J11, J2, J3, J4, J5, J6: Conn_01x01_Male, Connector_PinHeader_2.54mm:PinHeader_1x01_P2.54mm_Vertical, symbol Connector:Conn_01x01_Male
- added J10: Conn_01x04_Male, Connector_PinHeader_2.54mm:PinHeader_1x04_P2.54mm_Vertical, symbol Connector:Conn_01x04_Male
- added J12, J13, J9: Conn_01x02_Male, Connector_PinHeader_2.54mm:PinHeader_1x02_P2.54mm_Vertical, symbol Connector:Conn_01x02_Male
- added J8: Conn_01x03_Male, Connector_PinHeader_2.54mm:PinHeader_1x03_P2.54mm_Vertical, symbol Connector:Conn_01x03_Male
- added Q3: S8050, Package_TO_SOT_THT:TO-92_Inline, symbol Transistor_BJT:S8050
- added Q4: S8550, Package_TO_SOT_THT:TO-92_Inline, symbol Transistor_BJT:S8550
- added R31: 1K, Resistor_THT:R_Axial_DIN0207_L6.3mm_D2.5mm_P10.16mm_Horizontal, symbol Device:R
- C1, C3, C4: renamed from C?; footprint (none) -> Capacitor_THT:CP_Radial_D5.0mm_P2.00mm
- C12, C8: renamed from C?; value C -> 104; footprint (none) -> Capacitor_THT:C_Disc_D4.7mm_W2.5mm_P5.00mm
- C14, C15, C16, C17, C23, C24, C7: footprint (none) -> Capacitor_THT:C_Disc_D4.7mm_W2.5mm_P5.00mm
- C18, C19: value 103 -> 104; footprint (none) -> Capacitor_THT:C_Disc_D4.7mm_W2.5mm_P5.00mm
- C2: renamed from C?; footprint (none) -> Capacitor_THT:C_Disc_D4.7mm_W2.5mm_P5.00mm
- C20: value 102 -> 105; footprint (none) -> Capacitor_SMD:C_0805_2012Metric_Pad1.18x1.45mm_HandSolder
- C5, C6: footprint (none) -> Capacitor_SMD:C_0805_2012Metric_Pad1.18x1.45mm_HandSolder
- C9: renamed from C?; value C -> 105; footprint (none) -> Capacitor_SMD:C_0805_2012Metric_Pad1.18x1.45mm_HandSolder
- L9: footprint (none) -> Inductor_SMD:L_Taiyo-Yuden_MD-5050
- R1, R2, R25, R3, R5, R6, R7, R8: renamed from R?; footprint (none) -> Resistor_THT:R_Axial_DIN0207_L6.3mm_D2.5mm_P10.16mm_Horizontal
- R10, R9: value 2.5K -> 1K; footprint (none) -> Resistor_THT:R_Axial_DIN0207_L6.3mm_D2.5mm_P10.16mm_Horizontal
- R11, R12, R13, R14, R19, R20, R21, R22: value 22K -> 20K; footprint (none) -> Resistor_THT:R_Axial_DIN0207_L6.3mm_D2.5mm_P10.16mm_Horizontal
- R15, R16, R17, R18: value 10K -> 20K; footprint (none) -> Resistor_THT:R_Axial_DIN0207_L6.3mm_D2.5mm_P10.16mm_Horizontal
- R23, R24: value 500 -> 100; footprint (none) -> Resistor_THT:R_Axial_DIN0207_L6.3mm_D2.5mm_P10.16mm_Horizontal
- R26: value 100 -> 1K; footprint (none) -> Resistor_THT:R_Axial_DIN0207_L6.3mm_D2.5mm_P10.16mm_Horizontal
- R27, R4: footprint (none) -> Resistor_THT:R_Axial_DIN0207_L6.3mm_D2.5mm_P10.16mm_Horizontal
- R28: value 1K -> 100K; footprint (none) -> Resistor_THT:R_Axial_DIN0207_L6.3mm_D2.5mm_P10.16mm_Horizontal
- R29: value 22K -> 1K; footprint (none) -> Resistor_THT:R_Axial_DIN0207_L6.3mm_D2.5mm_P10.16mm_Horizontal
- R30: value 333 -> 1K; footprint (none) -> Resistor_THT:R_Axial_DIN0207_L6.3mm_D2.5mm_P10.16mm_Horizontal
- U2: renamed from U?; footprint (none) -> Package_DIP:DIP-8_W7.62mm
- U3: renamed from U?; footprint (none) -> Package_TO_SOT_SMD:SOT-223-3_TabPin2
- U6, U7: footprint (none) -> Package_DIP:DIP-14_W7.62mm
- U8: footprint (none) -> Package_DIP:DIP-8_W7.62mm
- Y1: footprint (none) -> Crystal:Crystal_HC49-4H_Vertical
- gave numbers to parts that had none: 1
Connections:
- net labels added: SPI1_MISO, SPI1_NSS
- net labels removed: +5V, -5V, COS+, COS-, SIN+, SIN-, SPI1_CS, SPWM, zheng_xian_bo
- wire segments 224 -> 225
- no-connect marks 1 -> 0
Other:
- note added: "shu_chu"
- note removed: "SPWM"
- note removed: "chuan_gan_qi"
- moved on the sheet: C9, U8B
