File: gcm0/citongmen/kacad/_autosave-fluxgate.sch (KiCad schematic (older format))
At the start: 105 parts, among them J1 +12, J11 SWD, J2 ji_li, Q1 BC547, Q10 KIA50N03, Q11 BC547, Q12 BC557, Q13 BC557, Q14 BC547, Q15 BC557, Q16 BC547, Q17 BC547, Q18 BC547, Q19 BC547, Q2 BC557, Q3 BC547, Q4 BC557, Q5 BC547, Q6 BC557, Q7 KIA50N03, Q8 KIA50N03, Q9 KIA50N03, U1 LM7809_TO220, U2 LM2596S-5, U3 LM7805_TO220, U4 TL084, U5 STM32F030F4P6, U6 LM1117-3.3, U9 74HC595, Y1 8M

Commit message: 电路改错
Parts:
- added Q? (x2): S8050, Package_TO_SOT_THT:TO-92_Inline, symbol Transistor_BJT:S8050
- added Q? (x2): S8550, Package_TO_SOT_THT:TO-92_Inline, symbol Transistor_BJT:S8550
Connections:
- net ji_li_0: now reaches C1.2, J2.1 (Pin_1), Q4.1 (C), Q7.3 (S), Q8.2 (D), R5.2, R9.2
- net ji_li_1: now reaches C3.2, J2.2 (Pin_2), Q10.2 (D), Q13.1 (C), Q9.3 (S), R13.2, R20.2
Changed lines of the file:
@@
 PA7_PWM1
-Wire Wire Line
-	9150 2750 9300 2750
-Wire Wire Line
-	9150 2000 9150 2750
-Connection ~ 9150 2750
-Wire Wire Line
-	9150 2750 9150 3650
 Wire Wire Line
 	1450 2000 1450 3650
@@
 $EndComp
 Wire Notes Line
-	500  8000 11750 8000
-Wire Notes Line
 	11750 8000 11750 11150
 Wire Notes Line
 	11750 11150 500  11150
-Wire Notes Line
-	500  11150 500  8000
 Wire Notes Line
 	8050 8000 8050 11150
@@
 Connection ~ 15150 5000
 Wire Wire Line
-	4700 3000 5250 3000
-Wire Wire Line
-	5350 3000 5900 3000
+	4700 3000 5100 3000
+Wire Wire Line
+	5350 3000 5600 3000
 $Comp
 L Device:C C?
@@
 Wire Wire Line
 	11200 6050 11650 6050
+Wire Notes Line
+	9800 3850 16000 3850
+Wire Notes Line
+	500  8000 16000 8000
+Wire Notes Line
+	9800 550  9800 8000
+Wire Notes Line
+	16000 550  16000 8000
+Wire Wire Line
+	9150 2000 9150 3650
+Wire Notes Line
+	500  550  500  11150
+Wire Notes Line
+	500  550  16000 550
+Wire Notes Line
+	500  4700 9800 4700
+Wire Wire Line
+	5100 3000 5100 2900
+Connection ~ 5100 3000
+Wire Wire Line
+	5100 3000 5250 3000
+Wire Wire Line
+	5600 3000 5600 2900
+Connection ~ 5600 3000
+Wire Wire Line
+	5600 3000 5900 3000
+Text Label 5100 2900 0    50   ~ 0
+ji_li_0
+Text Label 5600 2900 0    50   ~ 0
+ji_li_1
+$Comp
+L Transistor_BJT:S8050 Q?
+U 1 1 616E3B02
+P 3250 5500
+F 0 "Q?" H 3440 5546 50  0000 L CNN
+F 1 "S8050" H 3440 5455 50  0000 L CNN
+F 2 "Package_TO_SOT_THT:TO-92_Inline" H 3450 5425 50  0001 L CIN
+F 3 "http://www.unisonic.com.tw/datasheet/S8050.pdf" H 3250 5500 50  0001 L CNN
+	1    3250 5500
+	1    0    0    -1
+$EndComp
+$Comp
+L Transistor_BJT:S8050 Q?
+U 1 1 616E5340
+P 4900 5500
+F 0 "Q?" H 5090 5546 50  0000 L CNN
+F 1 "S8050" H 5090 5455 50  0000 L CNN
+F 2 "Package_TO_SOT_THT:TO-92_Inline" H 5100 5425 50  0001 L CIN
+F 3 "http://www.unisonic.com.tw/datasheet/S8050.pdf" H 4900 5500 50  0001 L CNN
+	1    4900 5500
+	1    0    0    -1
+$EndComp
+$Comp
+L Transistor_BJT:S8550 Q?
+U 1 1 616E6B8D
+P 3900 6200
+F 0 "Q?" H 4090 6246 50  0000 L CNN
+F 1 "S8550" H 4090 6155 50  0000 L CNN
+F 2 "Package_TO_SOT_THT:TO-92_Inline" H 4100 6125 50  0001 L CIN
+F 3 "http://www.unisonic.com.tw/datasheet/S8550.pdf" H 3900 6200 50  0001 L CNN
+	1    3900 6200
+	1    0    0    -1
+$EndComp
+$Comp
+L Transistor_BJT:S8550 Q?
+U 1 1 616E8316
+P 5150 6350
+F 0 "Q?" H 5340 6396 50  0000 L CNN
+F 1 "S8550" H 5340 6305 50  0000 L CNN
+F 2 "Package_TO_SOT_THT:TO-92_Inline" H 5350 6275 50  0001 L CIN
+F 3 "http://www.unisonic.com.tw/datasheet/S8550.pdf" H 5150 6350 50  0001 L CNN
+	1    5150 6350
+	1    0    0    -1
+$EndComp
 $EndSCHEMATC
