File: gcm0/citongmen/kacad/fluxgate.kicad_pcb (KiCad board)
At the start: 2 copper layers, 100 x 100 mm, 122 parts, among them J1 +12, J10 Conn_01x01_Male, J11 SWD, J12 Conn_01x01_Male, J2 Conn_01x01_Male, J3 Conn_01x01_Male, J4 Conn_01x01_Male, J5 Conn_01x01_Male, J6 GND, J7 Conn_01x01_Male, J8 Conn_01x01_Male, J9 Conn_01x01_Male, Q1 BC547, Q10 KIA50N03, Q11 BC547, Q12 BC557, Q13 BC557, Q14 BC547, Q15 BC557, Q16 BC547, Q17 BC547, Q18 BC547, Q19 BC547, Q2 BC557, Q20 S8050, Q21 S8550, Q22 S8050, Q23 S8550, Q3 BC547, Q4 BC557, Q5 BC547, Q6 BC557, Q7 KIA50N03, Q8 KIA50N03, Q9 KIA50N03, U2 LM2596S-5, U3 LM7805_TO220, U4 TL084, U5 STM32F030F4P6, U6 LM1117-3.3, U7 NE5532, U9 74HC595, Y1 8M

Commit message: PCB1
Routing:
- net -5V: track 302.2 -> 339.5 mm
- removed copper zone on F.Cu, net GND
Other:
- board text added: "+5"
- board text added: "-5"
- board text added: "A"
- board text added: "ADC"
- board text added: "B"
- board text added: "CLK"
- board text added: "DIO"
- board text added: "GND"
- board text added: "VCC"
