File: gcm0/lcr_1/kacad/lcr-1.kicad_pcb (KiCad board)
At the start: 2 copper layers, 100 x 100 mm, 119 parts, among them J1 -5V, J10 5V, J11 SWD, J12 -5V, J14 PA3, J15 SPWM, J16 PA9, J17 PA3, J18 PA9, J19 PA6, J2 Hc, J20 PA6, J21 PB1, J22 -5V, J23 5V, J24 3.3, J25 SPWM, J26 1.65V, J27 1.65V, J28 shuai_jian1, J29 shuan_jian, J3 Hp, J30 ADC, J31 +9V, J32 GND, J33 -5V, J34 5V, J35 3.3V, J36 shuai_jian1, J37 shuan_jian, J38 3.3V, J4 Lp, J5 Lc, J6 PB1, J7 5V, J8 5V, J9 ADC, Q1 BC547, Q2 BC547, Q3 BC547, SW1 SW_Push, SW2 SW_Push, U1 NE5532, U10 LM2596S-5, U2 STM32F030F4P6, U3 CD4053B, U4 CD4052B, U5 TL084, U6 LM358, U7 74HC595, U8 LM7805_TO220, U9 LM1117-3.3, Y1 8M

Commit message: PCB
Parts:
- removed the C12 at (172.4, 118.4)
- added C20: 105, Capacitor_SMD:C_0805_2012Metric_Pad1.18x1.45mm_HandSolder, F.Cu at (98.9, 95.4)
- added J10: Hc, Connector_Pin:Pin_D1.3mm_L11.0mm_LooseFit, F.Cu at (187.8, 132.0)
- added J11: Hp, Connector_Pin:Pin_D1.3mm_L11.0mm_LooseFit, F.Cu at (187.8, 136.7)
- added J6: Lc, Connector_Pin:Pin_D1.3mm_L11.0mm_LooseFit, F.Cu at (187.5, 152.1)
- added J9: Lp, Connector_Pin:Pin_D1.3mm_L11.0mm_LooseFit, F.Cu at (187.5, 147.5)
- added R19: 200, Resistor_THT:R_Axial_DIN0204_L3.6mm_D1.6mm_P2.54mm_Vertical, F.Cu at (172.2, 118.3)
- added R33: 100K, Resistor_THT:R_Axial_DIN0204_L3.6mm_D1.6mm_P2.54mm_Vertical, F.Cu at (106.7, 93.0)
- added R34: 100K, Resistor_THT:R_Axial_DIN0204_L3.6mm_D1.6mm_P2.54mm_Vertical, F.Cu at (113.0, 94.4)
- U8: footprint Package_TO_SOT_THT:TO-220-3_Horizontal_TabDown -> Package_TO_SOT_THT:TO-220-3_Vertical
- moved J23 48.9 mm to (152.8, 104.4)
- moved J24 48.9 mm to (150.7, 153.4)
- moved J3 2.41 mm to (182.8, 136.6)
- moved J4 2.26 mm to (182.9, 147.5)
- moved J5 2.19 mm to (183.0, 151.9)
- moved J2 1.99 mm to (183.2, 132.0)
- renumbered C13 to C12, C14 to C13, C15 to C14, C16 to C15, C17 to C16, C18 to C17, C19 to C18, C20 to C19, J38 to J12, J8 to J13, J9 to J14, J10 to J15, J11 to J16, J12 to J17, J14 to J18, J15 to J19, J16 to J20, J17 to J21, J18 to J22, J19 to J23, J20 to J24, J21 to J25, J22 to J26, J23 to J27, J24 to J28, J25 to J29, J26 to J30, J27 to J31, J28 to J32, J29 to J33, J30 to J34, J31 to J35, J32 to J36, J34 to J37, J35 to J38, J36 to J39, J37 to J40, J33 to J41, J6 to J7, J7 to J8, R19 to R20, R20 to R21, R21 to R22, R22 to R23, R23 to R24, R24 to R25, R25 to R26, R26 to R27, R27 to R28, R28 to R29, R29 to R30, R30 to R31, R31 to R32, R32 to R35, R33 to R36
Connections:
- DS1 pad : GND -> (no net)
- R30 pad 2: /PA5_SPI1_SCK_74HC595_11_SRCLK -> /PA4_SPI1_NSS_74HC595_12_RCLK
- R31 pad 2: /PA4_SPI1_NSS_74HC595_12_RCLK -> /PA5_SPI1_SCK_74HC595_11_SRCLK
- U10 pad 5: -5V -> Net-(R33-Pad1)
- U7 pad 11: /PA4_SPI1_NSS_74HC595_12_RCLK -> /PA5_SPI1_SCK_74HC595_11_SRCLK
- U7 pad 12: /PA5_SPI1_SCK_74HC595_11_SRCLK -> /PA4_SPI1_NSS_74HC595_12_RCLK
Routing:
- net +9V: track 45.6 -> 75.7 mm
- net Net-(R33-Pad1): track 0.00 -> 6.56 mm
- net Net-(C20-Pad1): track 0.00 -> 5.69 mm
- net /PA4_SPI1_NSS_74HC595_12_RCLK: track 61.2 -> 64.5 mm
- net -5V: track 125.4 -> 123.1 mm
- net /PA5_SPI1_SCK_74HC595_11_SRCLK: track 46.7 -> 45.2 mm, vias 0 -> 2
- net /Lc: track 79.7 -> 78.4 mm
- net /Lp: track 62.7 -> 61.5 mm
- net Net-(C21-Pad1): track 0.00 -> 1.05 mm
Other:
- board text added: "yjmwxwx_20210903"
- board text removed: "yjmwxwx_20210829"

Commit message: 调整档位
Parts:
- R17, R28: value 9K -> 20K
- R18, R27: value 1K -> 10K
