File: gcm0/lcr_5/kicad/lcr_2.kicad_pcb (KiCad board)
At the start: 2 copper layers, 100 x 100 mm, 226 parts, among them J1 5V, J2 -5V, J3 Conn_01x01_Male, J7 sin, Q1 BC547, Q2 BC547, Q3 BC547, SW1 1, SW2 2, SW3 SW_DIP_x01, U1 RC4580, U10 RC4580, U11 74HC595, U12 STM32F030F4P6, U13 L7809, U2 74HC4053PW,112, U3 74HC4052PW,118, U4 RC4580, U5 LM2596S-5, U6 LM7805_TO220, U7 RC4580, U8 LM1117-3.3, U9 74HC4053PW,112, Y1 8M

Commit message: 修改模拟电路
Parts:
- removed the J1 at (142.6, 80.6)
- removed the J1 at (132.6, 96.8)
- removed the J2 at (142.6, 84.0)
- removed the J2 at (130.8, 101.5)
- removed the J3 at (165.6, 78.3)
- removed the J3 at (136.7, 110.6)
- removed the J7 at (110.6, 52.4)
- removed the J7 at (175.9, 94.2)
- removed the REF** at (80.6, 99.2)
- removed the REF** at (154.2, 64.6)
- removed the REF** at (174.6, 116.5)
- removed the REF** at (162.4, 119.0)
- removed the REF** at (94.0, 119.5)
- removed the REF** at (102.5, 119.5)
- removed the REF** at (121.0, 119.5)
- removed the REF** at (131.0, 119.5)
- removed the REF** at (111.5, 119.5)
- removed the REF** at (141.5, 119.5)
- removed the REF** at (86.2, 118.7)
- removed the REF** at (80.6, 83.0)
- removed the REF** at (80.7, 118.7)
- removed the REF** at (151.5, 119.5)
- removed the REF** at (111.5, 128.6)
- removed the REF** at (86.2, 127.9)
- removed the REF** at (162.4, 128.1)
- removed the REF** at (131.0, 128.6)
- removed the REF** at (151.5, 128.6)
- removed the REF** at (102.5, 128.6)
- removed the REF** at (174.6, 125.6)
- removed the REF** at (94.0, 128.6)
- removed the REF** at (80.6, 93.7)
- removed the REF** at (121.0, 128.6)
- removed the REF** at (141.5, 128.6)
- removed the REF** at (80.8, 127.8)
- removed the REF** at (151.5, 137.5)
- removed the REF** at (174.6, 134.5)
- removed the REF** at (94.0, 137.5)
- removed the REF** at (102.5, 137.5)
- removed the REF** at (121.0, 137.5)
- removed the REF** at (80.7, 136.7)
- removed the REF** at (111.5, 137.5)
- removed the REF** at (94.5, 83.0)
- removed the REF** at (141.5, 137.5)
- removed the REF** at (86.2, 136.8)
- removed the REF** at (162.4, 137.0)
- removed the REF** at (131.0, 137.5)
- removed the REF** at (80.6, 61.7)
- removed the REF** at (80.6, 67.2)
- removed the REF** at (80.5, 77.9)
- removed the REF** at (86.2, 145.8)
- removed the REF** at (80.7, 145.7)
- removed the REF** at (151.5, 146.5)
- removed the REF** at (94.5, 109.9)
- removed the REF** at (141.5, 146.5)
- removed the REF** at (131.0, 146.5)
- removed the REF** at (121.0, 146.5)
- removed the REF** at (111.5, 146.5)
- removed the REF** at (102.5, 146.5)
- removed the REF** at (94.0, 146.5)
- removed the REF** at (174.6, 143.5)
- removed the REF** at (157.8, 65.8)
- removed the REF** at (154.4, 59.7)
- removed the REF** at (154.0, 61.7)
- removed the REF** at (80.6, 109.9)
- removed the REF** at (152.1, 61.8)
- removed the REF** at (144.7, 73.6)
- removed the REF** at (151.0, 73.7)
- removed the REF** at (149.6, 68.0)
- removed the REF** at (148.2, 64.7)
- removed the REF** at (144.7, 64.9)
- removed the REF** at (139.6, 62.9)
- removed the REF** at (136.8, 62.9)
- removed the REF** at (101.5, 74.5)
- removed the REF** at (103.4, 71.3)
- removed the REF** at (94.5, 51.0)
- removed the REF** at (111.5, 61.3)
- removed the REF** at (115.6, 61.8)
- removed the REF** at (113.3, 79.9)
- removed the REF** at (113.2, 77.8)
- removed the REF** at (120.4, 74.2)
- removed the REF** at (107.2, 83.9)
- removed the REF** at (118.7, 70.2)
- removed the REF** at (116.8, 72.4)
- removed the REF** at (175.3, 87.1)
- removed the REF** at (80.6, 51.0)
- removed the REF** at (99.7, 87.1)
- removed the REF** at (99.7, 81.8)
- removed the REF** at (175.3, 81.8)
- removed the REF** at (175.3, 51.1)
- removed the REF** at (99.7, 51.1)
- removed the REF** at (162.4, 146.0)
- removed the REF** at (129.1, 109.0)
- removed the REF** at (176.4, 104.0)
- removed the REF** at (173.2, 104.0)
- removed the REF** at (170.3, 104.0)
- removed the REF** at (94.5, 77.9)
- removed the REF** at (167.4, 104.0)
- removed the REF** at (150.8, 108.8)
- removed the REF** at (147.1, 105.1)
- removed the REF** at (167.1, 108.6)
- removed the REF** at (154.4, 109.3)
- removed the REF** at (150.6, 113.7)
- removed the REF** at (152.9, 113.7)
- removed the REF** at (155.2, 113.7)
- added C48: 106, Capacitor_SMD:C_0805_2012Metric_Pad1.18x1.45mm_HandSolder, F.Cu at (163.9, 105.2)
- added D11: 1N4007, Diode_THT:D_DO-41_SOD81_P2.54mm_Vertical_AnodeUp, F.Cu at (102.3, 77.0)
- added D12: 1N4007, Diode_THT:D_DO-41_SOD81_P2.54mm_Vertical_AnodeUp, F.Cu at (105.8, 79.5)
- added D13: 1N4007, Diode_THT:D_DO-41_SOD81_P2.54mm_Vertical_AnodeUp, F.Cu at (102.2, 73.4)
- added D14: 1N4007, Diode_THT:D_DO-41_SOD81_P2.54mm_Vertical_AnodeUp, F.Cu at (105.9, 71.1)
- added J1: 5V, Connector_PinHeader_2.54mm:PinHeader_1x01_P2.54mm_Vertical, F.Cu at (125.7, 108.0)
- added J1: 5V, Connector_PinHeader_2.54mm:PinHeader_1x01_P2.54mm_Vertical, F.Cu at (149.0, 56.4)
- added J2: -5V, Connector_PinHeader_2.54mm:PinHeader_1x01_P2.54mm_Vertical, F.Cu at (127.4, 98.8)
- added J2: -5V, Connector_PinHeader_2.54mm:PinHeader_1x01_P2.54mm_Vertical, F.Cu at (137.5, 85.3)
- added J3: Conn_01x01_Male, Connector_PinHeader_2.54mm:PinHeader_1x01_P2.54mm_Vertical, F.Cu at (137.6, 76.5)
- added J4: SWD, Connector_PinHeader_2.54mm:PinHeader_1x03_P2.54mm_Vertical, B.Cu at (111.8, 84.4)
- added J7: sin, Connector_PinHeader_2.54mm:PinHeader_1x01_P2.54mm_Vertical, F.Cu at (112.8, 89.4)
- added J7: sin, Connector_PinHeader_2.54mm:PinHeader_1x01_P2.54mm_Vertical, F.Cu at (108.0, 85.2)
- added R29: 20K, Resistor_SMD:R_0805_2012Metric_Pad1.20x1.40mm_HandSolder, F.Cu at (105.0, 110.4)
- added R31: 20K, Resistor_SMD:R_0805_2012Metric_Pad1.20x1.40mm_HandSolder, F.Cu at (121.0, 111.1)
- added R33: 100, Resistor_SMD:R_0805_2012Metric_Pad1.20x1.40mm_HandSolder, F.Cu at (136.8, 116.5)
- added R34: 1K, Resistor_SMD:R_0805_2012Metric_Pad1.20x1.40mm_HandSolder, F.Cu at (132.1, 111.2)
- added R36: 1K, Resistor_SMD:R_0805_2012Metric_Pad1.20x1.40mm_HandSolder, F.Cu at (141.7, 112.6)
- added R38: 900, Resistor_SMD:R_0805_2012Metric_Pad1.20x1.40mm_HandSolder, F.Cu at (144.8, 100.4)
- added R39: 100, Resistor_SMD:R_0805_2012Metric_Pad1.20x1.40mm_HandSolder, F.Cu at (144.8, 104.3)
- added R40: 100, Resistor_SMD:R_0805_2012Metric_Pad1.20x1.40mm_HandSolder, F.Cu at (142.2, 89.7)
- added R41: 500, Resistor_SMD:R_0805_2012Metric_Pad1.20x1.40mm_HandSolder, F.Cu at (145.1, 91.1)
- added R53: 10K, Resistor_SMD:R_0805_2012Metric_Pad1.20x1.40mm_HandSolder, F.Cu at (160.8, 106.3)
- added R54: 20K, Resistor_SMD:R_0805_2012Metric_Pad1.20x1.40mm_HandSolder, F.Cu at (167.7, 111.4)
- added R55: 10K, Resistor_SMD:R_0805_2012Metric_Pad1.20x1.40mm_HandSolder, F.Cu at (168.6, 108.3)
- added R56: 100, Resistor_SMD:R_0805_2012Metric_Pad1.20x1.40mm_HandSolder, F.Cu at (99.2, 102.4)
- added R57: 100, Resistor_SMD:R_0805_2012Metric_Pad1.20x1.40mm_HandSolder, F.Cu at (99.1, 107.4)
- added REF**: TestPoint_Pad_D1.5mm, TestPoint:TestPoint_Pad_D1.5mm, F.Cu at (167.5, 102.2)
- added REF**: Pin_D0.7mm_L6.5mm_W1.8mm_FlatFork, Connector_Pin:Pin_D0.7mm_L6.5mm_W1.8mm_FlatFork, F.Cu at (172.6, 92.4)
- added REF**: 2.25, Connector_Pin:2.25, F.Cu at (84.0, 81.0)
- added REF**: 2.25, Connector_Pin:2.25, F.Cu at (97.5, 81.0)
- added REF**: 2.25, Connector_Pin:2.25, F.Cu at (97.5, 50.5)
- added REF**: 2.25, Connector_Pin:2.25, F.Cu at (84.0, 50.5)
- added REF**: 2.25, Connector_Pin:2.25, F.Cu at (86.5, 71.0)
- added REF**: 2.25, Connector_Pin:2.25, F.Cu at (86.5, 65.0)
- added REF**: 2.25, Connector_Pin:2.25, F.Cu at (180.7, 84.0)
- added REF**: 2.25, Connector_Pin:2.25, F.Cu at (178.2, 50.5)
- added REF**: 2.25, Connector_Pin:2.25, F.Cu at (103.2, 50.5)
- added REF**: Pin_D0.7mm_L6.5mm_W1.8mm_FlatFork, Connector_Pin:Pin_D0.7mm_L6.5mm_W1.8mm_FlatFork, F.Cu at (143.6, 118.9)
- added REF**: Pin_D0.7mm_L6.5mm_W1.8mm_FlatFork, Connector_Pin:Pin_D0.7mm_L6.5mm_W1.8mm_FlatFork, F.Cu at (154.9, 117.7)
- added REF**: Pin_D0.7mm_L6.5mm_W1.8mm_FlatFork, Connector_Pin:Pin_D0.7mm_L6.5mm_W1.8mm_FlatFork, F.Cu at (160.7, 98.6)
- added REF**: Pin_D0.7mm_L6.5mm_W1.8mm_FlatFork, Connector_Pin:Pin_D0.7mm_L6.5mm_W1.8mm_FlatFork, F.Cu at (159.9, 101.0)
- added REF**: Pin_D0.7mm_L6.5mm_W1.8mm_FlatFork, Connector_Pin:Pin_D0.7mm_L6.5mm_W1.8mm_FlatFork, F.Cu at (157.1, 101.3)
- added REF**: TestPoint_Pad_D1.5mm, TestPoint:TestPoint_Pad_D1.5mm, F.Cu at (148.6, 100.8)
- added REF**: TestPoint_Pad_D1.5mm, TestPoint:TestPoint_Pad_D1.5mm, F.Cu at (147.9, 96.9)
- added REF**: TestPoint_Pad_D1.5mm, TestPoint:TestPoint_Pad_D1.5mm, F.Cu at (149.6, 95.7)
- added REF**: TestPoint_Pad_D1.5mm, TestPoint:TestPoint_Pad_D1.5mm, F.Cu at (149.6, 93.4)
- added REF**: TestPoint_Pad_D1.5mm, TestPoint:TestPoint_Pad_D1.5mm, F.Cu at (164.0, 101.2)
- added REF**: TestPoint_Pad_D1.5mm, TestPoint:TestPoint_Pad_D1.5mm, F.Cu at (152.5, 92.3)
- added REF**: TestPoint_Pad_D1.5mm, TestPoint:TestPoint_Pad_D1.5mm, F.Cu at (131.0, 120.5)
- added REF**: TestPoint_Pad_D1.5mm, TestPoint:TestPoint_Pad_D1.5mm, F.Cu at (130.5, 115.8)
- added REF**: Pin_D0.7mm_L6.5mm_W1.8mm_FlatFork, Connector_Pin:Pin_D0.7mm_L6.5mm_W1.8mm_FlatFork, F.Cu at (113.2, 121.3)
- added REF**: TestPoint_Pad_D1.5mm, TestPoint:TestPoint_Pad_D1.5mm, F.Cu at (116.7, 111.4)
- added REF**: TestPoint_Pad_D1.5mm, TestPoint:TestPoint_Pad_D1.5mm, F.Cu at (106.6, 113.1)
- added REF**: TestPoint_Pad_D1.5mm, TestPoint:TestPoint_Pad_D1.5mm, F.Cu at (106.9, 116.7)
- added REF**: TestPoint_Pad_D1.5mm, TestPoint:TestPoint_Pad_D1.5mm, F.Cu at (118.9, 112.2)
- added REF**: TestPoint_Pad_D1.5mm, TestPoint:TestPoint_Pad_D1.5mm, F.Cu at (120.9, 106.8)
- added REF**: Pin_D0.7mm_L6.5mm_W1.8mm_FlatFork, Connector_Pin:Pin_D0.7mm_L6.5mm_W1.8mm_FlatFork, F.Cu at (118.3, 109.5)
- added REF**: TestPoint_Pad_D1.5mm, TestPoint:TestPoint_Pad_D1.5mm, F.Cu at (170.5, 103.6)
- added REF**: Pin_D0.7mm_L6.5mm_W1.8mm_FlatFork, Connector_Pin:Pin_D0.7mm_L6.5mm_W1.8mm_FlatFork, F.Cu at (115.6, 109.5)
- added REF**: TestPoint_Pad_D1.5mm, TestPoint:TestPoint_Pad_D1.5mm, F.Cu at (117.5, 101.0)
- added REF**: TestPoint_Pad_D1.5mm, TestPoint:TestPoint_Pad_D1.5mm, F.Cu at (118.1, 95.5)
- added REF**: TestPoint_Pad_2.0x2.0mm, TestPoint:TestPoint_Pad_2.0x2.0mm, F.Cu at (116.0, 89.6)
- added REF**: TestPoint_Pad_2.0x2.0mm, TestPoint:TestPoint_Pad_2.0x2.0mm, F.Cu at (110.6, 97.8)
- added REF**: Pin_D0.7mm_L6.5mm_W1.8mm_FlatFork, Connector_Pin:Pin_D0.7mm_L6.5mm_W1.8mm_FlatFork, F.Cu at (132.0, 84.5)
- added REF**: Pin_D0.7mm_L6.5mm_W1.8mm_FlatFork, Connector_Pin:Pin_D0.7mm_L6.5mm_W1.8mm_FlatFork, F.Cu at (131.7, 80.5)
- added REF**: Pin_D0.7mm_L6.5mm_W1.8mm_FlatFork, Connector_Pin:Pin_D0.7mm_L6.5mm_W1.8mm_FlatFork, F.Cu at (129.8, 80.5)
- added REF**: Pin_D0.7mm_L6.5mm_W1.8mm_FlatFork, Connector_Pin:Pin_D0.7mm_L6.5mm_W1.8mm_FlatFork, F.Cu at (127.9, 80.5)
- added REF**: TestPoint_Pad_D1.5mm, TestPoint:TestPoint_Pad_D1.5mm, F.Cu at (154.8, 106.6)
- added REF**: Pin_D0.7mm_L6.5mm_W1.8mm_FlatFork, Connector_Pin:Pin_D0.7mm_L6.5mm_W1.8mm_FlatFork, F.Cu at (126.1, 66.8)
- added REF**: Pin_D0.7mm_L6.5mm_W1.8mm_FlatFork, Connector_Pin:Pin_D0.7mm_L6.5mm_W1.8mm_FlatFork, F.Cu at (127.9, 69.7)
- added REF**: Pin_D0.7mm_L6.5mm_W1.8mm_FlatFork, Connector_Pin:Pin_D0.7mm_L6.5mm_W1.8mm_FlatFork, F.Cu at (129.7, 69.7)
- added REF**: Pin_D0.7mm_L6.5mm_W1.8mm_FlatFork, Connector_Pin:Pin_D0.7mm_L6.5mm_W1.8mm_FlatFork, F.Cu at (125.2, 80.0)
- added REF**: Pin_D0.7mm_L6.5mm_W1.8mm_FlatFork, Connector_Pin:Pin_D0.7mm_L6.5mm_W1.8mm_FlatFork, F.Cu at (126.1, 69.7)
- added REF**: 2.25, Connector_Pin:2.25, F.Cu at (105.8, 120.6)
- added REF**: 2.25, Connector_Pin:2.25, F.Cu at (180.7, 120.6)
- added REF**: 2.25, Connector_Pin:2.25, F.Cu at (178.2, 87.0)
- added REF**: 2.25, Connector_Pin:2.25, F.Cu at (103.3, 87.1)
- added REF**: 2.25, Connector_Pin:2.25, F.Cu at (105.7, 84.1)
- added REF**: TestPoint_Pad_D1.5mm, TestPoint:TestPoint_Pad_D1.5mm, F.Cu at (131.6, 57.3)
- added REF**: PinHeader_1x01_P2.54mm_Vertical, Connector_PinHeader_2.54mm:PinHeader_1x01_P2.54mm_Vertical, F.Cu at (149.1, 127.1)
- added REF**: PinHeader_1x01_P2.54mm_Vertical, Connector_PinHeader_2.54mm:PinHeader_1x01_P2.54mm_Vertical, F.Cu at (118.5, 127.2)
- added REF**: PinHeader_1x01_P2.54mm_Vertical, Connector_PinHeader_2.54mm:PinHeader_1x01_P2.54mm_Vertical, F.Cu at (129.3, 127.2)
- added REF**: 2.25, Connector_Pin:2.25, F.Cu at (173.9, 125.3)
- added REF**: Pin_D0.9mm_L10.0mm_W2.4mm_FlatFork, Connector_Pin:Pin_D0.9mm_L10.0mm_W2.4mm_FlatFork, F.Cu at (179.8, 125.1)
- added REF**: PinHeader_1x01_P2.54mm_Vertical, Connector_PinHeader_2.54mm:PinHeader_1x01_P2.54mm_Vertical, F.Cu at (108.3, 127.3)
- added REF**: PinHeader_1x01_P2.54mm_Vertical, Connector_PinHeader_2.54mm:PinHeader_1x01_P2.54mm_Vertical, F.Cu at (159.3, 127.2)
- added REF**: 2.25, Connector_Pin:2.25, F.Cu at (89.2, 125.2)
- added REF**: PinHeader_1x01_P2.54mm_Vertical, Connector_PinHeader_2.54mm:PinHeader_1x01_P2.54mm_Vertical, F.Cu at (138.8, 127.1)
- added REF**: PinHeader_1x01_P2.54mm_Vertical, Connector_PinHeader_2.54mm:PinHeader_1x01_P2.54mm_Vertical, F.Cu at (98.8, 127.3)
- added REF**: TestPoint_Pad_D1.5mm, TestPoint:TestPoint_Pad_D1.5mm, F.Cu at (141.6, 66.9)
- added REF**: 2.25, Connector_Pin:2.25, F.Cu at (83.8, 125.1)
- added REF**: PinHeader_1x01_P2.54mm_Vertical, Connector_PinHeader_2.54mm:PinHeader_1x01_P2.54mm_Vertical, F.Cu at (98.8, 133.8)
- added REF**: PinHeader_1x01_P2.54mm_Vertical, Connector_PinHeader_2.54mm:PinHeader_1x01_P2.54mm_Vertical, F.Cu at (159.3, 133.7)
- added REF**: PinHeader_1x01_P2.54mm_Vertical, Connector_PinHeader_2.54mm:PinHeader_1x01_P2.54mm_Vertical, F.Cu at (118.6, 133.7)
- added REF**: PinHeader_1x01_P2.54mm_Vertical, Connector_PinHeader_2.54mm:PinHeader_1x01_P2.54mm_Vertical, F.Cu at (108.3, 133.8)
- added REF**: 2.25, Connector_Pin:2.25, F.Cu at (83.8, 131.6)
- added REF**: 2.25, Connector_Pin:2.25, F.Cu at (89.3, 131.7)
- added REF**: 2.25, Connector_Pin:2.25, F.Cu at (174.0, 131.8)
- added REF**: Pin_D0.9mm_L10.0mm_W2.4mm_FlatFork, Connector_Pin:Pin_D0.9mm_L10.0mm_W2.4mm_FlatFork, F.Cu at (179.9, 131.6)
- added REF**: PinHeader_1x01_P2.54mm_Vertical, Connector_PinHeader_2.54mm:PinHeader_1x01_P2.54mm_Vertical, F.Cu at (149.1, 133.6)
- added REF**: TestPoint_Pad_D1.5mm, TestPoint:TestPoint_Pad_D1.5mm, F.Cu at (138.4, 64.9)
- added REF**: PinHeader_1x01_P2.54mm_Vertical, Connector_PinHeader_2.54mm:PinHeader_1x01_P2.54mm_Vertical, F.Cu at (129.4, 133.7)
- added REF**: PinHeader_1x01_P2.54mm_Vertical, Connector_PinHeader_2.54mm:PinHeader_1x01_P2.54mm_Vertical, F.Cu at (138.9, 133.6)
- added REF**: PinHeader_1x01_P2.54mm_Vertical, Connector_PinHeader_2.54mm:PinHeader_1x01_P2.54mm_Vertical, F.Cu at (118.6, 140.2)
- added REF**: PinHeader_1x01_P2.54mm_Vertical, Connector_PinHeader_2.54mm:PinHeader_1x01_P2.54mm_Vertical, F.Cu at (138.9, 140.1)
- added REF**: PinHeader_1x01_P2.54mm_Vertical, Connector_PinHeader_2.54mm:PinHeader_1x01_P2.54mm_Vertical, F.Cu at (98.8, 140.3)
- added REF**: 2.25, Connector_Pin:2.25, F.Cu at (89.3, 138.2)
- added REF**: 2.25, Connector_Pin:2.25, F.Cu at (174.0, 138.3)
- added REF**: PinHeader_1x01_P2.54mm_Vertical, Connector_PinHeader_2.54mm:PinHeader_1x01_P2.54mm_Vertical, F.Cu at (129.3, 140.2)
- added REF**: 2.25, Connector_Pin:2.25, F.Cu at (83.8, 138.1)
- added REF**: PinHeader_1x01_P2.54mm_Vertical, Connector_PinHeader_2.54mm:PinHeader_1x01_P2.54mm_Vertical, F.Cu at (108.3, 140.3)
- added REF**: TestPoint_Pad_D1.5mm, TestPoint:TestPoint_Pad_D1.5mm, F.Cu at (134.0, 65.4)
- added REF**: PinHeader_1x01_P2.54mm_Vertical, Connector_PinHeader_2.54mm:PinHeader_1x01_P2.54mm_Vertical, F.Cu at (159.3, 140.2)
- added REF**: PinHeader_1x01_P2.54mm_Vertical, Connector_PinHeader_2.54mm:PinHeader_1x01_P2.54mm_Vertical, F.Cu at (149.1, 140.1)
- added REF**: Pin_D0.9mm_L10.0mm_W2.4mm_FlatFork, Connector_Pin:Pin_D0.9mm_L10.0mm_W2.4mm_FlatFork, F.Cu at (179.8, 138.1)
- added REF**: 2.25, Connector_Pin:2.25, F.Cu at (174.0, 144.8)
- added REF**: PinHeader_1x01_P2.54mm_Vertical, Connector_PinHeader_2.54mm:PinHeader_1x01_P2.54mm_Vertical, F.Cu at (159.3, 146.7)
- added REF**: PinHeader_1x01_P2.54mm_Vertical, Connector_PinHeader_2.54mm:PinHeader_1x01_P2.54mm_Vertical, F.Cu at (129.3, 146.7)
- added REF**: PinHeader_1x01_P2.54mm_Vertical, Connector_PinHeader_2.54mm:PinHeader_1x01_P2.54mm_Vertical, F.Cu at (149.1, 146.6)
- added REF**: PinHeader_1x01_P2.54mm_Vertical, Connector_PinHeader_2.54mm:PinHeader_1x01_P2.54mm_Vertical, F.Cu at (138.8, 146.7)
- added REF**: PinHeader_1x01_P2.54mm_Vertical, Connector_PinHeader_2.54mm:PinHeader_1x01_P2.54mm_Vertical, F.Cu at (118.6, 146.7)
- added REF**: PinHeader_1x01_P2.54mm_Vertical, Connector_PinHeader_2.54mm:PinHeader_1x01_P2.54mm_Vertical, F.Cu at (108.3, 146.8)
- added REF**: Pin_D0.7mm_L6.5mm_W1.8mm_FlatFork, Connector_Pin:Pin_D0.7mm_L6.5mm_W1.8mm_FlatFork, F.Cu at (172.3, 118.8)
- added REF**: 2.25, Connector_Pin:2.25, F.Cu at (89.2, 144.7)
- added REF**: Pin_D0.9mm_L10.0mm_W2.4mm_FlatFork, Connector_Pin:Pin_D0.9mm_L10.0mm_W2.4mm_FlatFork, F.Cu at (179.8, 144.6)
- added REF**: 2.25, Connector_Pin:2.25, F.Cu at (83.8, 144.6)
- added REF**: PinHeader_1x01_P2.54mm_Vertical, Connector_PinHeader_2.54mm:PinHeader_1x01_P2.54mm_Vertical, F.Cu at (98.8, 146.8)
- added REF**: 2.25, Connector_Pin:2.25, F.Cu at (86.5, 102.0)
- added REF**: 2.25, Connector_Pin:2.25, F.Cu at (84.0, 118.0)
- added REF**: 2.25, Connector_Pin:2.25, F.Cu at (97.5, 118.0)
- added REF**: 2.25, Connector_Pin:2.25, F.Cu at (84.0, 87.5)
- added REF**: 2.25, Connector_Pin:2.25, F.Cu at (86.5, 108.0)
- added REF**: 2.25, Connector_Pin:2.25, F.Cu at (97.5, 87.5)
- C1, C11, C12, C16, C18, C19, C24, C25, C26, C29, C30, C32, C33, C34, C36, C37, C38, C4, C40, C41, C42, C43, C44, C5, C6, C7, C8, C9: footprint Capacitor_SMD:C_0603_1608Metric_Pad1.08x0.95mm_HandSolder -> Capacitor_SMD:C_0805_2012Metric_Pad1.18x1.45mm_HandSolder
- C10, C13: value 204 -> 2uF; footprint Capacitor_SMD:C_0603_1608Metric_Pad1.08x0.95mm_HandSolder -> Capacitor_SMD:C_0805_2012Metric_Pad1.18x1.45mm_HandSolder
- C15: value 104 -> 106; footprint Capacitor_SMD:C_0603_1608Metric_Pad1.08x0.95mm_HandSolder -> Capacitor_SMD:C_0805_2012Metric_Pad1.18x1.45mm_HandSolder
- C17: footprint Capacitor_SMD:C_0603_1608Metric_Pad1.08x0.95mm_HandSolder -> Capacitor_SMD:C_0805_2012Metric_Pad1.18x1.45mm_HandSolder; moved to F.Cu
- C2: value 104 -> 204; footprint Capacitor_SMD:C_0603_1608Metric_Pad1.08x0.95mm_HandSolder -> Capacitor_SMD:C_0805_2012Metric_Pad1.18x1.45mm_HandSolder
- C22, C27, C31, REF**: moved to F.Cu
- C47: value 10 -> 15; footprint Capacitor_SMD:C_0603_1608Metric_Pad1.08x0.95mm_HandSolder -> Capacitor_SMD:C_0805_2012Metric_Pad1.18x1.45mm_HandSolder
- R1: value 50 -> 100; footprint Resistor_THT:R_Axial_DIN0204_L3.6mm_D1.6mm_P1.90mm_Vertical -> Resistor_SMD:R_0805_2012Metric_Pad1.20x1.40mm_HandSolder
- R10, R11, R12, R13, R14, R15, R16, R19, R2, R20, R21, R22, R25, R28, R3, R30, R32, R35, R37, R4, R42, R43, R44, R45, R46, R47, R48, R49, R50, R51, R52, R7, R8, R9: footprint Resistor_THT:R_Axial_DIN0204_L3.6mm_D1.6mm_P1.90mm_Vertical -> Resistor_SMD:R_0805_2012Metric_Pad1.20x1.40mm_HandSolder
- R17: value 1K -> 10K; footprint Resistor_THT:R_Axial_DIN0204_L3.6mm_D1.6mm_P1.90mm_Vertical -> Resistor_SMD:R_0805_2012Metric_Pad1.20x1.40mm_HandSolder
- R18: value 100K -> 10K; footprint Resistor_THT:R_Axial_DIN0204_L3.6mm_D1.6mm_P1.90mm_Vertical -> Resistor_SMD:R_0805_2012Metric_Pad1.20x1.40mm_HandSolder
- R23, R24: value 2K -> 1K; footprint Resistor_THT:R_Axial_DIN0204_L3.6mm_D1.6mm_P1.90mm_Vertical -> Resistor_SMD:R_0805_2012Metric_Pad1.20x1.40mm_HandSolder
- R26, R27: value 10K -> 1K; footprint Resistor_THT:R_Axial_DIN0204_L3.6mm_D1.6mm_P1.90mm_Vertical -> Resistor_SMD:R_0805_2012Metric_Pad1.20x1.40mm_HandSolder
- R5, R6: value 100 -> 20K
- U1, U10, U4, U7: value RC4580 -> MC4580G-S08-R
- moved D8 95.0 mm to (179.2, 59.7), turned to 90 degrees
- moved C4 90.7 mm to (176.1, 59.1)
- moved D9 81.1 mm to (173.2, 61.1), turned to 270 degrees
- moved C5 78.0 mm to (101.8, 66.2)
- moved BT1 76.0 mm to (165.4, 67.2), turned to 0 degrees
- moved U13 76.0 mm to (173.8, 72.3), turned to 270 degrees
- moved C10 74.9 mm to (104.6, 66.2)
- moved Q1 74.4 mm to (103.7, 62.1)
- moved SW3 71.8 mm to (169.7, 62.4)
- moved C19 71.4 mm to (168.7, 67.3), turned to 270 degrees
- moved DS1 71.3 mm to (108.7, 53.0), turned to 90 degrees
- moved C42 70.9 mm to (115.5, 70.9), turned to 90 degrees
- moved C3 70.6 mm to (110.3, 71.7), turned to 270 degrees
- moved R10 69.8 mm to (110.1, 75.6), turned to 0 degrees
- moved Y1 68.2 mm to (119.5, 72.1), turned to 270 degrees
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Connections:
- R27 pad 1: Net-(C14-Pad2) -> Net-(R27-Pad1)
- R32 pad 1: Net-(R32-Pad1) -> /4053_1
- R37 pad 2: Net-(C15-Pad2) -> Net-(R37-Pad2)
- R5 pad 1: /HC -> Net-(R5-Pad1)
- R5 pad 2: /HP -> /LP
- R6 pad 1: /LP -> Net-(R6-Pad1)
- R6 pad 2: /LC -> /HP
- SW1 pad : (no net) -> GND
- SW2 pad : (no net) -> GND
- U10 pad 1: Net-(C15-Pad2) -> Net-(R37-Pad2)
- U10 pad 2: Net-(U10-Pad2) -> Net-(R35-Pad1)
- U10 pad 3: Net-(R32-Pad1) -> Net-(C48-Pad1)
- U10 pad 6: Net-(U10-Pad6) -> Net-(R21-Pad1)
- U2 pad 1: Net-(U2-Pad1) -> Net-(R31-Pad1)
- U2 pad 2: /HP -> Net-(R6-Pad1)
- U2 pad 3: /LC -> Net-(R29-Pad1)
- U2 pad 5: /LP -> Net-(R5-Pad1)
- U3 pad 13: Net-(U2-Pad1) -> Net-(R31-Pad2)
- U4 pad 2: Net-(R23-Pad2) -> Net-(R33-Pad2)
- U4 pad 6: Net-(R24-Pad2) -> Net-(R33-Pad1)
- U7 pad 1: Net-(R32-Pad1) -> /4053_1
- U7 pad 2: Net-(U7-Pad2) -> Net-(R30-Pad2)
- U7 pad 7: Net-(C14-Pad2) -> Net-(R27-Pad1)
- U9 pad 1: Net-(R35-Pad1) -> /4053_1
- U9 pad 12: /ADC -> Net-(R54-Pad2)
- U9 pad 13: Net-(R21-Pad1) -> Net-(R37-Pad2)
- U9 pad 14: Net-(U10-Pad6) -> Net-(C15-Pad2)
- U9 pad 15: Net-(U10-Pad2) -> Net-(C48-Pad2)
- U9 pad 2: Net-(C15-Pad2) -> /4053_2
- U9 pad 3: Net-(R30-Pad2) -> Net-(R27-Pad1)
- U9 pad 4: Net-(U7-Pad2) -> Net-(C14-Pad2)
- U9 pad 5: Net-(R32-Pad1) -> Net-(R38-Pad2)
Routing:
- net (no net): track 0.00 -> 60.8 mm
- net Net-(R32-Pad1): track 48.0 -> 0.00 mm
- net Net-(R37-Pad2): track 0.00 -> 36.4 mm
- net /CLK: track 3.49 -> 29.7 mm
- net GND: track 159.6 -> 184.8 mm, vias 44 -> 161
- net Net-(U10-Pad6): track 24.6 -> 0.00 mm, vias 2 -> 0
- net Net-(C15-Pad2): track 39.9 -> 15.4 mm, vias 1 -> 0
- net Net-(U10-Pad2): track 23.9 -> 0.00 mm
- net /DIO: track 6.05 -> 29.1 mm
- net Net-(R35-Pad1): track 29.7 -> 8.05 mm, vias 1 -> 0
- net Net-(U2-Pad4): track 12.5 -> 34.1 mm
- net Net-(R54-Pad2): track 0.00 -> 20.8 mm
- net Net-(U2-Pad1): track 20.1 -> 0.00 mm
- net Net-(R27-Pad1): track 0.00 -> 19.1 mm, vias 0 -> 2
- net Net-(U7-Pad2): track 18.2 -> 0.00 mm
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Other:
- board text added: "3.3V"
- board text added: "GND"
- board text added: "SWD"
- board text removed: "BOOT"
- board text removed: "BT1"
- board text removed: "SPWM"
- board text removed: "SW3"
