File: gcm0/nei_zu_yi/kicad/nei_zu_yi.sch (KiCad schematic (older format))
At the start: 150 parts, among them J1 LC, J2 HC, J3 LP, J4 Conn_01x01_Male, J5 SWD, J6 HP, Q1 Q_NMOS_GDS, Q2 Q_NMOS_GDS, Q3 SS8050, Q4 SS8550, Q5 SS8050, Q6 SS8550, SW1 SW_Push, SW2 SW_Push, U1 CD4053B, U11 74HC595, U12 STM32F030F4P6, U2 TL084, U3 TL084, U4 NE5532, U5 CD4053B, U6 LM2596S-5, U7 LM7805_TO220, U9 LM1117-3.3, Y1 8M

Commit message: 修改KICAD原理图标注错误
Parts:
- gave numbers to parts that had none: 4
- renumbered C15 to C1, C19 to C10, C23 to C11, C45 to C12, C14 to C13, C11 to C14, C8 to C15, C5 to C16, C18 to C17, C13 to C18, C20 to C19, C38 to C2, C25 to C20, C27 to C21, C39 to C22, C6 to C23, C1 to C24, C2 to C25, C43 to C26, C44 to C27, C4 to C28, C9 to C29, C17 to C3, C21 to C30, C42 to C31, C10 to C32, C22 to C33, C40 to C34, C41 to C35, C33 to C36, C26 to C37, C37 to C38, C34 to C39, C24 to C4, C35 to C40, C32 to C41, C16 to C42, C36 to C43, C28 to C44, C3 to C45, C12 to C46, C29 to C5, C30 to C6, D4 to D1, D8 to D10, D5 to D2, D7 to D3, D1 to D4, D2 to D5, D3 to D6, D9 to D7, D10 to D8, D6 to D9, J4 to J1, J6 to J3, J5 to J4, J1 to J5, J3 to J6, Q3 to Q1, Q5 to Q2, Q4 to Q3, Q6 to Q4, Q1 to Q5, Q2 to Q6, R10 to R1, R64 to R10, R3 to R11, R8 to R12, R4 to R13, R9 to R14, R19 to R15, R21 to R16, R11 to R17, R12 to R19, R14 to R20, R22 to R21, R5 to R22, R1 to R23, R6 to R25, R2 to R26, R65 to R27, R7 to R28, R17 to R29, R34 to R3, R16 to R30, R50 to R31, R23 to R32, R28 to R33, R46 to R34, R57 to R36, R59 to R37, R61 to R38, R44 to R39, R37 to R4, R51 to R40, R32 to R41, R36 to R42, R58 to R43, R62 to R44, R63 to R45, R25 to R46, R29 to R47, R45 to R48, R33 to R49, R40 to R5, R38 to R50, R41 to R51, R56 to R53, R60 to R54, R39 to R55, R55 to R56, R26 to R57, R30 to R58, R27 to R59, R42 to R6, R15 to R60, R13 to R61, R53 to R62, R54 to R63, R47 to R64, R48 to R65, R49 to R66, R31 to R7, R18 to R8, R20 to R9, U2 to U1, U3 to U1, U11 to U10, U9 to U2, U7 to U3, U6 to U4, U1 to U5, U4 to U6, U3 to U7, U2 to U7, U12 to U8, U5 to U9
